Commit message: creted world file

File: description/lidar.xacro (robot description, xacro)
@@ -26,5 +26,5 @@
         <sensor name="laser" type="ray">
             <pose> 0 0 0 0 0 0 </pose>
-            <visualize>true</visualize>
+            <visualize>false</visualize>
             <update_rate>7</update_rate>
             <ray>

File: description/robot_core.xacro (robot description, xacro)
@@ -139,5 +139,5 @@
         <parent link="chassis"/>
         <child link="actuator_body"/>
-        <origin xyz="0.32 0 0.01" rpy="0 0 0"/>
+        <origin xyz="0.28 0 0.01" rpy="0 0 0"/>
     </joint>
     <link name="actuator_body">
@@ -150,5 +150,5 @@
         </visual>
         <collision>
-            <origin xyz="0.0075 0 0" rpy="-1.571 0 3.14"/>
+            <origin xyz="0.0 0.0075 0.0" rpy="-1.571 0 3.14"/>
             <geometry>
                 <mesh filename="file://$(find arms_bot)/meshes/actuator_body.stl" scale="1.0 1.0 1.0"/>
@@ -172,5 +172,5 @@
     <link name="actuator_rod">
         <visual>
-            <origin xyz="0 0 0.29" rpy=" -1.5708 0 0"/>
+            <origin xyz="0 0 0.30" rpy=" -1.5708 0 0"/>
             <geometry>
               <mesh filename="file://$(find arms_bot)/meshes/actuator_rod.stl" scale="1.0 1.0 1.0"/>
@@ -179,5 +179,5 @@
         </visual>
         <collision>
-            <origin xyz="0 0 0.29" rpy=" -1.5708 0 0"/>
+            <origin xyz="0 0 0.30" rpy=" -1.5708 0 0"/>
             <geometry>
                 <mesh filename="file://$(find arms_bot)/meshes/actuator_rod.stl" scale="1.0 1.0 1.0"/>
@@ -185,5 +185,5 @@
         </collision>
         <xacro:inertial_cylinder mass="0.3" length="0.25" radius="0.01">
-            <origin xyz="0 0 0.29" rpy=" -1.5708 0 0"/>
+            <origin xyz="0 0 0.30" rpy=" -1.5708 0 0"/>
         </xacro:inertial_cylinder>
     </link>
