Commit message: added camera

File: description/robot.urdf.xacro (robot description, xacro)
@@ -4,3 +4,4 @@
     <xacro:include filename="gazebo_control.xacro"/>
     <xacro:include filename="lidar.xacro"/>
+    <xacro:include filename="camera.xacro"/>
 </robot>

File: description/robot_core.xacro (robot description, xacro)
@@ -25,4 +25,7 @@
     <material name="brown">
         <color rgba="0.6 0.4 0.2 1"/>
+    </material>
+    <material name="green">
+         <color rgba="0 1 0 1"/>
     </material>
     <!-- BASE LINK -->
