Commit message: Add gazebo control plugin and update URDF files for robot description

File: description/robot_core.xacro (robot description, xacro)
@@ -23,4 +23,7 @@
       <color rgba="0.75 0.75 0.75 1"/>
     </material>
+    <material name="brown">
+        <color rgba="0.6 0.4 0.2 1"/>
+    </material>
     <!-- BASE LINK -->
     <link name="base_link">
@@ -50,4 +53,7 @@
         </xacro:inertial_box>
     </link>
+    <gazebo reference="chassis">
+        <material>Gazebo/White</material>
+    </gazebo>
     <!-- LEFT WHEEL LINK -->
     <joint name="left_wheel_joint" type="continuous">
@@ -73,4 +79,7 @@
         </xacro:inertial_cylinder>
     </link>
+    <gazebo reference="left_wheel">
+        <material>Gazebo/Yellow</material>
+    </gazebo>
     <!-- RIGHT WHEEL LINK -->
     <joint name="right_wheel_joint" type="continuous">
@@ -96,4 +105,7 @@
         </xacro:inertial_cylinder>
     </link>
+    <gazebo reference="right_wheel">
+        <material>Gazebo/Yellow</material>
+    </gazebo>
     <!-- CASTER WHEEL LINK -->
     <joint name="caster_wheel_joint" type="fixed">
@@ -118,4 +130,9 @@
         </xacro:inertial_sphere>
     </link>
+    <gazebo reference="caster_wheel">
+        <material>Gazebo/Black</material>
+        <mu1 value="0.001"/>
+        <mu2 value="0.001"/>
+    </gazebo>
     <!-- ACTUATOR_BODY LINK -->
     <joint name="actuator_body_joint" type="fixed">
@@ -142,4 +159,7 @@
         </xacro:inertial_cylinder>
     </link>
+    <gazebo reference="actuator_body">
+        <material>Gazebo/Black</material>
+    </gazebo>
         <!-- ACTUATOR_ROD LINK -->
     <joint name="actuator_rod_joint" type="prismatic">
@@ -168,4 +188,7 @@
         </xacro:inertial_cylinder>
     </link>
+    <gazebo reference="actuator_rod">
+        <material>Gazebo/Silver</material>
+    </gazebo>
        <!-- FORKLIFT LINK -->
     <joint name="forklift_joint" type="fixed">
@@ -180,5 +203,5 @@
               <mesh filename="file://$(find arms_bot)/meshes/forklift.stl" scale="1.0 1.0 1.0"/>
             </geometry>
-            <material name="silver"/>
+            <material name="brown"/>
         </visual>
         <collision>
@@ -192,3 +215,6 @@
         </xacro:inertial_box>
     </link>
+    <gazebo reference="forklift">
+        <material>Gazebo/Orange</material>
+    </gazebo>
 </robot>

Commit message: minor fixes

File: description/robot_core.xacro (robot description, xacro)
@@ -75,5 +75,5 @@
         <collision>
             <geometry>
-                <cylinder radius="0.05" length="0.026"/>
+                <sphere radius="0.05"/>
             </geometry>
         </collision>
@@ -101,5 +101,5 @@
         <collision>
             <geometry>
-                <cylinder radius="0.05" length="0.026"/>
+                <sphere radius="0.05"/>
             </geometry>
         </collision>
@@ -126,5 +126,5 @@
         <collision>
             <geometry>
-                <mesh filename="file://$(find arms_bot)/meshes/caster_wheel.stl" scale="1.0 1.0 1.0"/>
+                <sphere radius="0.016"/>
             </geometry>
         </collision>
@@ -142,5 +142,5 @@
         <parent link="chassis"/>
         <child link="actuator_body"/>
-        <origin xyz="0.28 0 0.01" rpy="0 0 0"/>
+        <origin xyz="0.28 0 0.02" rpy="0 0 0"/>
     </joint>
     <link name="actuator_body">
@@ -167,13 +167,13 @@
         <!-- ACTUATOR_ROD LINK -->
     <joint name="actuator_rod_joint" type="prismatic">
-        <parent link="actuator_body"/>
+        <parent link="base_link"/>
         <child link="actuator_rod"/>
-        <origin xyz="0.0 0 0.0" rpy="0 0 0"/>
+        <origin xyz="0.2 0 0.09" rpy="0 0 0"/>
         <axis xyz="0 0 1"/>
-        <limit lower="0.0" upper="0.2" effort="1500" velocity="0.007"/>
+        <limit lower="0.0" upper="0.2" effort="1000" velocity="0.007"/>
     </joint>
     <link name="actuator_rod">
         <visual>
-            <origin xyz="0 0 0.30" rpy=" -1.5708 0 0"/>
+            <origin xyz="0 0 0.225" rpy=" -1.571 0 0"/>
             <geometry>
               <mesh filename="file://$(find arms_bot)/meshes/actuator_rod.stl" scale="1.0 1.0 1.0"/>
@@ -182,5 +182,5 @@
         </visual>
         <collision>
-            <origin xyz="0 0 0.30" rpy=" -1.5708 0 0"/>
+            <origin xyz="0 0 0.225" rpy=" -1.5708 0 0"/>
             <geometry>
                 <mesh filename="file://$(find arms_bot)/meshes/actuator_rod.stl" scale="1.0 1.0 1.0"/>
@@ -188,5 +188,5 @@
         </collision>
         <xacro:inertial_cylinder mass="0.3" length="0.25" radius="0.01">
-            <origin xyz="0 0 0.30" rpy=" -1.5708 0 0"/>
+            <origin xyz="0 0 0.225" rpy=" -1.5708 0 0"/>
         </xacro:inertial_cylinder>
     </link>
@@ -198,9 +198,9 @@
         <parent link="actuator_rod"/>
         <child link="forklift"/>
-        <origin xyz="0.014 0 0.273" rpy="0 0 0"/>
+        <origin xyz="0.014 0 0.208" rpy="0 0 0"/>
     </joint>
     <link name="forklift">
         <visual>
-            <origin xyz="0 0 0" rpy=" 0 0 1.5708"/>
+            <origin xyz=" 0 0 0" rpy=" 0 0 1.5708"/>
             <geometry>
               <mesh filename="file://$(find arms_bot)/meshes/forklift.stl" scale="1.0 1.0 1.0"/>
